Commit message: build

File: src/articubot_one/description/robot_all.xacro (robot description, xacro)
@@ -179,5 +179,5 @@
                 <cylinder radius="${caster_wheel_radius}" length="${caster_wheel_thickness}" />
             </geometry>
-        <material name="white" />
+        <material name="whiste" />
         </visual>
         <collision>
